Commit message: t265Slam

File: linorobot2/linorobot2_description/urdf/controllers/diff_drive.urdf.xacro (robot description, xacro)
@@ -4,5 +4,5 @@
       <plugin name="differential_drive_controller" filename="libgazebo_ros_diff_drive.so">
         <ros>
-          <argument>odom:=odom/unfiltered</argument>
+          <argument>odom:=camera/pose/sample</argument>
         </ros>
         <updateRate>100</updateRate>

File: linorobot2/linorobot2_description/urdf/mech/base.urdf.xacro (robot description, xacro)
@@ -38,4 +38,9 @@
       </visual>
     </gazebo>
+    <!-- <joint name="base_to_footprint" type="fixed">
+      <parent link="base_footprint"/>
+      <child link="base_link"/>
+      <origin xyz="0 0 ${wheel_radius - wheel_pos_z}" rpy="0 0 0"/>
+    </joint> -->
     <joint name="base_to_footprint" type="fixed">
       <parent link="base_footprint"/>

File: linorobot2/linorobot2_description/urdf/sensors/laser.urdf.xacro (robot description, xacro)
@@ -36,6 +36,11 @@
       </visual>
     </gazebo>
-    <joint name="${frame_id}_to_base_link" type="fixed">
+    <!-- <joint name="${frame_id}_to_base_link" type="fixed">
       <parent link="base_link"/>
+      <child link="${frame_id}"/>
+      <xacro:insert_block name="origin" />
+    </joint> -->
+    <joint name="${frame_id}_to_camera_link" type="fixed">
+      <parent link="camera_link"/>
       <child link="${frame_id}"/>
       <xacro:insert_block name="origin" />
